File: hardware/board/tang_nano_hat.kicad_pcb (KiCad board)
At the start: 2 copper layers, 70 x 26 mm, 27 parts, among them J1 Conn_01x24, J2 Conn_01x24, J3 AF SS-JB17.6, U1 SN74LVC2G17DBVR, U2 TPD2EUSB30ADRTR, U3 AP2151DWG-7

Commit message: feat: logo
Parts:
- added G***: LOGO, LOGO, F.Cu at (114.3, 62.7)
Routing:
- net KEYBOARD_VBUS: track 18.7 -> 49.4 mm, vias 1 -> 2
- net GND: vias 79 -> 83

Commit message: feat: mounting holes
Parts:
- added H1: MountingHole, MountingHole:MountingHole_2.2mm_M2, F.Cu at (167.3, 52.6)
- added H2: MountingHole, MountingHole:MountingHole_2.2mm_M2, F.Cu at (167.3, 73.4)
- moved D1 0.40 mm to (140.4, 67.5)
- moved R2 0.40 mm to (135.9, 67.7)
- moved C1 0.40 mm to (138.2, 68.3)
- moved R1 0.40 mm to (138.2, 66.8)
- moved R3 0.40 mm to (138.2, 69.8)
- moved R10 0.21 mm to (145.8, 66.8)
- moved R9 0.21 mm to (145.8, 68.3)
Routing:
- net KEYBOARD_VBUS: track 49.4 -> 18.7 mm, vias 2 -> 1
- net /33: track 26.3 -> 29.0 mm
- net GND: vias 83 -> 82

Commit message: rfac
Other:
- board text added: "woldhack 2026"

Commit message: feat: cool silkscreen
Parts:
- added G***: LOGO, LOGO, B.Cu at (131.0, 62.4)
- R10: value 100K -> 3.9K
